Commit message: sim: run user's Lightning-LM and Nav2 on the simulated robots
- lightning.launch.py: sim replaces only the sensor drivers; mapping and
  localization use lightning's g1_online.launch.py and navigation uses
  aid_navigation2's navigation2.launch.py + nav2_params.yaml, rewritten at
  launch time for Humble, sim time and the simulated robot's size
- livox_bridge: PointCloud2 -> livox_ros_driver2/CustomMsg on /livox/lidar
  (raw CDR, verified by round-tripping through deserialize_message)
- sim.launch.py: stack:=standalone|lightning; lightning stack roots the URDF
  at body_link and leaves map->base_link to Lightning
- install.sh: MPPI and STVL plugins; README: Lightning workflow and results

File: sim_ws/src/robot_nav_sim/urdf/ackermann_car.urdf.xacro (robot description, xacro)
@@ -21,11 +21,11 @@
   <material name="car_orange"><color rgba="0.86 0.45 0.14 1"/></material>
   <material name="deck_grey"><color rgba="0.30 0.31 0.33 1"/></material>
-  <link name="base_footprint"/>
+  <link name="${root}"/>
   <joint name="base_joint" type="fixed">
-    <parent link="base_footprint"/>
-    <child link="base_link"/>
+    <parent link="${root}"/>
+    <child link="${trunk}"/>
     <origin xyz="0 0 ${body_z}" rpy="0 0 0"/>
   </joint>
-  <link name="base_link">
+  <link name="${trunk}">
     <inertial>
       <origin xyz="${body_cx} 0 0"/>
@@ -49,12 +49,12 @@
   </link>
   <!-- 后轮（驱动） -->
-  <xacro:drive_wheel name="rear_left_wheel"  parent="base_link" xyz="0 ${track / 2} ${wheel_r - body_z}"
+  <xacro:drive_wheel name="rear_left_wheel"  parent="${trunk}" xyz="0 ${track / 2} ${wheel_r - body_z}"
                      radius="${wheel_r}" width="${wheel_w}" mass="0.8"/>
-  <xacro:drive_wheel name="rear_right_wheel" parent="base_link" xyz="0 ${-track / 2} ${wheel_r - body_z}"
+  <xacro:drive_wheel name="rear_right_wheel" parent="${trunk}" xyz="0 ${-track / 2} ${wheel_r - body_z}"
                      radius="${wheel_r}" width="${wheel_w}" mass="0.8"/>
   <!-- 前轮：转向节（绕 z 轴）+ 车轮（自由滚动） -->
   <xacro:macro name="steer_wheel" params="side ly">
     <joint name="front_${side}_steer_joint" type="revolute">
-      <parent link="base_link"/>
+      <parent link="${trunk}"/>
       <child link="front_${side}_steer"/>
       <origin xyz="${wheel_base} ${ly * kingpin / 2} ${wheel_r - body_z}" rpy="0 0 0"/>
@@ -74,5 +74,5 @@
   <xacro:steer_wheel side="right" ly="-1"/>
   <!-- Mid-360 装在车顶前部 -->
-  <xacro:mid360 parent="base_link" xyz="${wheel_base} 0 ${body_t / 2 + 0.085}"/>
+  <xacro:mid360 parent="${trunk}" xyz="${wheel_base} 0 ${body_t / 2 + 0.085}"/>
   <gazebo>
     <!-- 阿克曼转向：订阅 /robot/cmd_vel（Twist，按 v 和 w 换算前轮转角），发布里程计 -->
@@ -95,5 +95,5 @@
       <tf_topic>/robot/tf</tf_topic>
       <frame_id>odom</frame_id>
-      <child_frame_id>base_footprint</child_frame_id>
+      <child_frame_id>${root}</child_frame_id>
       <odom_publish_frequency>50</odom_publish_frequency>
     </plugin>

File: sim_ws/src/robot_nav_sim/urdf/common.xacro (robot description, xacro)
@@ -2,4 +2,11 @@
 <!-- 三台机器人共用的部分：Mid-360 雷达 + IMU、关节状态、仿真真值。话题名对三台机器人都一样。 -->
 <robot xmlns:xacro="http://www.ros.org/wiki/xacro">
+  <!-- 坐标系名。默认 base_footprint（脚下）/ base_link（躯干），配合本包自带的 Nav2。
+       接 Lightning-LM 时改成 root_link:=body_link trunk_link:=trunk：
+       Lightning 自己发布 map->base_link->body_link 和 base_link->base_footprint，URDF 里不能再出现这两个名字。 -->
+  <xacro:arg name="root_link" default="base_footprint"/>
+  <xacro:arg name="trunk_link" default="base_link"/>
+  <xacro:property name="root" value="$(arg root_link)"/>
+  <xacro:property name="trunk" value="$(arg trunk_link)"/>
   <material name="lidar_black"><color rgba="0.08 0.08 0.09 1"/></material>
   <!--
@@ -83,5 +90,5 @@
       <plugin filename="gz-sim-odometry-publisher-system" name="gz::sim::systems::OdometryPublisher">
         <odom_frame>world</odom_frame>
-        <robot_base_frame>base_footprint</robot_base_frame>
+        <robot_base_frame>${root}</robot_base_frame>
         <odom_topic>/robot/ground_truth</odom_topic>
         <tf_topic>/robot/ground_truth/tf</tf_topic>
@@ -107,5 +114,5 @@
         <tf_topic>/robot/tf</tf_topic>
         <frame_id>odom</frame_id>
-        <child_frame_id>base_footprint</child_frame_id>
+        <child_frame_id>${root}</child_frame_id>
         <odom_publish_frequency>50</odom_publish_frequency>
       </plugin>
@@ -130,5 +137,5 @@
         <tf_topic>/robot/tf</tf_topic>
         <frame_id>odom</frame_id>
-        <child_frame_id>base_footprint</child_frame_id>
+        <child_frame_id>${root}</child_frame_id>
         <odom_publish_frequency>50</odom_publish_frequency>
       </plugin>

File: sim_ws/src/robot_nav_sim/urdf/diff_car.urdf.xacro (robot description, xacro)
@@ -13,11 +13,11 @@
   <material name="car_blue"><color rgba="0.16 0.36 0.62 1"/></material>
   <material name="deck_grey"><color rgba="0.30 0.31 0.33 1"/></material>
-  <link name="base_footprint"/>
+  <link name="${root}"/>
   <joint name="base_joint" type="fixed">
-    <parent link="base_footprint"/>
-    <child link="base_link"/>
+    <parent link="${root}"/>
+    <child link="${trunk}"/>
     <origin xyz="0 0 ${body_z}" rpy="0 0 0"/>
   </joint>
-  <link name="base_link">
+  <link name="${trunk}">
     <inertial>
       <mass value="12.0"/>
@@ -37,12 +37,12 @@
     </collision>
   </link>
-  <xacro:drive_wheel name="left_wheel"  parent="base_link" xyz="0 ${wheel_sep / 2} ${wheel_r - body_z}"
+  <xacro:drive_wheel name="left_wheel"  parent="${trunk}" xyz="0 ${wheel_sep / 2} ${wheel_r - body_z}"
                      radius="${wheel_r}" width="${wheel_w}"/>
-  <xacro:drive_wheel name="right_wheel" parent="base_link" xyz="0 ${-wheel_sep / 2} ${wheel_r - body_z}"
+  <xacro:drive_wheel name="right_wheel" parent="${trunk}" xyz="0 ${-wheel_sep / 2} ${wheel_r - body_z}"
                      radius="${wheel_r}" width="${wheel_w}"/>
-  <xacro:caster name="front_caster" parent="base_link" xyz="0.19 0 ${0.035 - body_z}" radius="0.035" visible="true"/>
-  <xacro:caster name="rear_caster"  parent="base_link" xyz="-0.19 0 ${0.035 - body_z}" radius="0.035" visible="true"/>
+  <xacro:caster name="front_caster" parent="${trunk}" xyz="0.19 0 ${0.035 - body_z}" radius="0.035" visible="true"/>
+  <xacro:caster name="rear_caster"  parent="${trunk}" xyz="-0.19 0 ${0.035 - body_z}" radius="0.035" visible="true"/>
   <!-- Mid-360 装在车顶中间 -->
-  <xacro:mid360 parent="base_link" xyz="0.10 0 ${body_t / 2 + 0.085}"/>
+  <xacro:mid360 parent="${trunk}" xyz="0.10 0 ${body_t / 2 + 0.085}"/>
   <xacro:diff_drive_plugin separation="${wheel_sep}" radius="${wheel_r}" max_v="1.0" max_w="2.0"/>
   <xacro:common_plugins/>

File: sim_ws/src/robot_nav_sim/urdf/go2.urdf.xacro (robot description, xacro)
@@ -19,11 +19,11 @@
   <material name="body_grey"><color rgba="0.82 0.83 0.85 1"/></material>
   <material name="leg_dark"><color rgba="0.20 0.21 0.23 1"/></material>
-  <link name="base_footprint"/>
+  <link name="${root}"/>
   <joint name="base_joint" type="fixed">
-    <parent link="base_footprint"/>
-    <child link="base_link"/>
+    <parent link="${root}"/>
+    <child link="${trunk}"/>
     <origin xyz="0 0 ${body_h}" rpy="0 0 0"/>
   </joint>
-  <link name="base_link">
+  <link name="${trunk}">
     <inertial>
       <!-- 质心故意放低到离地约 0.13 m：隐藏底盘轴距短（为了能原地转），
@@ -49,5 +49,5 @@
   <xacro:macro name="leg" params="name fx ly hip_rpy thigh_mesh calf_mesh">
     <joint name="${name}_hip_joint" type="fixed">
-      <parent link="base_link"/>
+      <parent link="${trunk}"/>
       <child link="${name}_hip"/>
       <origin xyz="${fx * 0.1934} ${ly * 0.0465} 0" rpy="0 0 0"/>
@@ -126,14 +126,14 @@
        0.8 仍远大于爬 25° 坡需要的 tan(25°)≈0.47。 -->
   <xacro:property name="wheel_x" value="0.12"/>
-  <xacro:drive_wheel name="front_left_wheel"  parent="base_link" xyz="${wheel_x} ${wheel_sep / 2} ${wheel_r - body_h}"
+  <xacro:drive_wheel name="front_left_wheel"  parent="${trunk}" xyz="${wheel_x} ${wheel_sep / 2} ${wheel_r - body_h}"
                      radius="${wheel_r}" width="0.04" visible="false" mu="0.8"/>
-  <xacro:drive_wheel name="front_right_wheel" parent="base_link" xyz="${wheel_x} ${-wheel_sep / 2} ${wheel_r - body_h}"
+  <xacro:drive_wheel name="front_right_wheel" parent="${trunk}" xyz="${wheel_x} ${-wheel_sep / 2} ${wheel_r - body_h}"
                      radius="${wheel_r}" width="0.04" visible="false" mu="0.8"/>
-  <xacro:drive_wheel name="rear_left_wheel"   parent="base_link" xyz="${-wheel_x} ${wheel_sep / 2} ${wheel_r - body_h}"
+  <xacro:drive_wheel name="rear_left_wheel"   parent="${trunk}" xyz="${-wheel_x} ${wheel_sep / 2} ${wheel_r - body_h}"
                      radius="${wheel_r}" width="0.04" visible="false" mu="0.8"/>
-  <xacro:drive_wheel name="rear_right_wheel"  parent="base_link" xyz="${-wheel_x} ${-wheel_sep / 2} ${wheel_r - body_h}"
+  <xacro:drive_wheel name="rear_right_wheel"  parent="${trunk}" xyz="${-wheel_x} ${-wheel_sep / 2} ${wheel_r - body_h}"
                      radius="${wheel_r}" width="0.04" visible="false" mu="0.8"/>
   <!-- Mid-360 装在机身前上方 -->
-  <xacro:mid360 parent="base_link" xyz="0.19 0 0.105"/>
+  <xacro:mid360 parent="${trunk}" xyz="0.19 0 0.105"/>
   <!-- 滑移转向的等效轮距：原地转时轮子打滑，实际转得比运动学少（实测约 0.73 倍），
        所以插件里的轮距按 0.36 / 0.73 ≈ 0.49 标定，让 cmd_vel 和里程计的角速度都对得上 -->
